File: PCB-Business-Card.kicad_pcb (KiCad board)
At the start: 2 copper layers, 91 x 55 mm, 43 parts, among them J2 GPIO Breakout, U1 ESP32-C3FH4, U3 USBLC6-2SC6, U4 AMS1117-3.3, Y1 L327S400H11L

Commit message: Final Tapeout Version
Parts:
- added C19: 150pF, Capacitor_SMD:C_0402_1005Metric_Pad0.74x0.62mm_HandSolder, F.Cu at (82.8, 55.5)
- added C20: 100nF, Capacitor_SMD:C_0402_1005Metric, F.Cu at (86.2, 50.2)
- added U2: NT3H2111W0FHKH, C710403:C710403, F.Cu at (86.2, 52.2)
- J1: renamed from USB C
- renumbered 2.4GHz to AE1, RESET to SW1, BOOT to SW2
Connections:
- U1 pad 19: Net-(U1-SPIHD) -> unconnected-(U1-SPIHD-Pad19)
- U1 pad 20: Net-(U1-SPIWP) -> unconnected-(U1-SPIWP-Pad20)
- U1 pad 21: /SPICS0 -> unconnected-(U1-SPICS0-Pad21)
- U1 pad 22: Net-(U1-SPICLK) -> unconnected-(U1-SPICLK-Pad22)
- U1 pad 23: Net-(U1-SPID) -> unconnected-(U1-SPID-Pad23)
- U1 pad 24: Net-(U1-SPIQ) -> unconnected-(U1-SPIQ-Pad24)
Routing:
- net Net-(U2-LA): track 0.00 -> 371.4 mm, vias 0 -> 2
- net Net-(J1-D--PadA7): track 34.7 -> 51.9 mm, vias 2 -> 3
- net /VBUS: track 63.1 -> 74.9 mm, vias 4 -> 5
- net Net-(J1-D+-PadA6): track 31.4 -> 38.5 mm, vias 1 -> 2
- net GND: track 67.4 -> 74.4 mm, vias 52 -> 55
- net Net-(U2-LB): track 0.00 -> 4.31 mm
- net Net-(U2-VOUT): track 0.00 -> 1.41 mm
- net Net-(J1-CC1): track 18.3 -> 19.0 mm
Other:
- board text added: "2.4GHz"
- board text added: "BOOT"
- board text added: "D+"
- board text added: "D-"
- board text added: "RESET"
- board text added: "VBUS"

Commit message: Added README and firmware
Connections:
- C16 pad 1: +3V3 -> +3.3V
- D1 pad 2: +3V3 -> +3.3V
- J2 pad 2: +3V3 -> +3.3V
- R3 pad 1: +3V3 -> +3.3V
- R4 pad 1: +3V3 -> +3.3V
- R6 pad 2: +3V3 -> +3.3V
- R7 pad 2: +3V3 -> +3.3V
- U4 pad 2: +3V3 -> +3.3V
Routing:
- net +3.3V: track 26.4 -> 137.2 mm, vias 2 -> 14
- net +3V3: track 109.2 -> 0.00 mm, vias 12 -> 0
