File: PCB-Business-Card.kicad_sch (KiCad schematic)
At the start: 43 parts, among them J1 USB C, J2 GPIO Breakout, SW1 RESET, SW2 BOOT, U1 ESP32-C3FH4, U3 USBLC6-2SC6, U4 AMS1117-3.3, Y1 L327S400H11L

Commit message: Final Tapeout Version
Parts:
- added AE2: PCB Antenna, symbol Device:Antenna_Loop
- added C19: 150pF, Capacitor_SMD:C_0402_1005Metric_Pad0.74x0.62mm_HandSolder, symbol Device:C
- added C20: 100nF, Capacitor_SMD:C_0402_1005Metric, symbol Device:C
- added U2: NT3H2111W0FHKH, C710403:C710403, symbol C710403:NT3H2111W0FHKH
- AE1: now left out of the parts list
Connections:
- net GND: now also C20.2, U2.2 (VSS)
- new net: AE2.1, C19.1, U2.1 (LA)
- new net: AE2.2, C19.2, U2.8 (LB)
- new net: C20.1, U2.7 (VOUT)
Other:
- note added: "NFC Antenna"
- note removed: "Flash (If not using ESP32-C3FH4)"

Commit message: Added README and firmware
Connections:
- net +3V3 is gone; now on net +3.3V: C16.1, D1.2 (A), J2.2 (Pin_2), R3.1, R4.1, R6.2, R7.2, U4.2 (VO)
Changed lines of the file:
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@@
 	(wire
 		(pts
+			(xy 106.68 27.94) (xy 114.3 27.94)
+		)
+		(stroke
+			(width 0)
+			(type default)
+		)
+	)
+	(wire
+		(pts
 			(xy 119.38 83.82) (xy 128.27 83.82)
 		)
@@
 	)
 	(symbol
+		(lib_id "power:+3.3V")
+		(at 114.3 27.94 270)
+		(unit 1)
+		(exclude_from_sim no)
+		(in_bom yes)
+		(on_board yes)
+		(dnp no)
+		(property "Reference" "#PWR036"
+			(at 110.49 27.94 0)
+			(effects
+				(font
+					(size 1.27 1.27)
+				)
+				(hide yes)
+			)
+		)
+		(property "Value" "+3.3V"
+			(at 119.38 27.94 90)
+			(effects
+				(font
+					(size 1.27 1.27)
+				)
+			)
+		)
+		(property "Footprint" ""
+			(at 114.3 27.94 0)
+			(effects
+				(font
+					(size 1.27 1.27)
+				)
+				(hide yes)
+			)
+		)
+		(property "Datasheet" ""
+			(at 114.3 27.94 0)
+			(effects
+				(font
+					(size 1.27 1.27)
+				)
+				(hide yes)
+			)
+		)
+		(property "Description" "Power symbol creates a global label with name \"+3.3V\""
+			(at 114.3 27.94 0)
+			(effects
+				(font
+					(size 1.27 1.27)
+				)
+				(hide yes)
+			)
+		)
+		(pin "1"
+		)
+		(instances
+			(project "PCB-Business-Card"
+				(path "/0ca6a2bc-2c3c-484d-be7e-ed2eceee1aef"
+					(reference "#PWR036")
+					(unit 1)
+				)
+			)
+		)
+	)
+	(symbol
 		(lib_id "power:GND")
 		(at 163.83 40.64 90)
@@
 					(unit 1)
 				)
+			)
+		)
+	)
+	(symbol
+		(lib_id "power:+3V3")
+		(at 106.68 27.94 90)
+		(unit 1)
+		(exclude_from_sim no)
+		(in_bom yes)
+		(on_board yes)
+		(dnp no)
+		(property "Reference" "#PWR035"
+			(at 110.49 27.94 0)
+			(effects
+				(font
+					(size 1.27 1.27)
+				)
+				(hide yes)
+			)
+		)
+		(property "Value" "+3V3"
+			(at 101.6 27.94 90)
+			(effects
+				(font
+					(size 1.27 1.27)
+				)
+			)
+		)
+		(property "Footprint" ""
+			(at 106.68 27.94 0)
+			(effects
+				(font
+					(size 1.27 1.27)
+				)
+				(hide yes)
+			)
+		)
+		(property "Datasheet" ""
+			(at 106.68 27.94 0)
+			(effects
+				(font
+					(size 1.27 1.27)
+				)
+				(hide yes)
+			)
+		)
+		(property "Description" "Power symbol creates a global label with name \"+3V3\""
+			(at 106.68 27.94 0)
+			(effects
+				(font
+					(size 1.27 1.27)
+				)
+				(hide yes)
+			)
+		)
+		(pin "1"
+		)
+		(instances
+			(project "PCB-Business-Card"
+				(path "/0ca6a2bc-2c3c-484d-be7e-ed2eceee1aef"
+					(reference "#PWR035")
+					(unit 1)
+				)
